File: Eagle/Arduinoboy.brd (EAGLE design)
At the start: 68.6 x 53.3 mm, 20 parts

Commit message: update eagle files
Parts:
- removed R3: 2k, SparkFun-Resistors:AXIAL-0.3
- removed U$1: GBA-LINK, David:GBA-LINK
- added U$4: GBA-LINK, Catskulls_link_port:GBA-LINK
- moved R1 2.54 mm to (16.9, 42.4)
- moved R2 2.54 mm to (14.3, 42.4)
- moved R4 2.54 mm to (21.9, 42.4)
- moved R5 2.54 mm to (19.4, 42.4)
Connections:
- removed net N$18: U$1.VCC, U$3.VIN
- removed net N$4: R3.P$2, S2.1, S2.2, U$3.D3
- new net N$20: S2.1, S2.2, U$3.D2
- new net PS2_CLK: U$3.D3, X1.5
- new net PS2_DATA: U$3.D7, X1.1
- new net VIN: U$3.VIN
- net GND: now also S2.3, S2.4, U$4.GND; no longer R3.P$1, U$1.GND
- net N$17: now also U$4.SC; no longer U$1.SC, X1.5
- net N$21: now also U$4.SO; no longer U$1.SO, X1.1
- net N$22: now also U$4.SI; no longer U$1.SI
- net VCC: now also U$4.SD, U$4.VCC; no longer S2.3, S2.4
Routing:
- net N$4: track 128.5 -> 0.00 mm
- net N$20: track 0.00 -> 87.0 mm, vias 0 -> 2
- net PS2_DATA: track 0.00 -> 71.5 mm
- net PS2_CLK: track 0.00 -> 57.7 mm, vias 0 -> 1
- net N$18: track 48.3 -> 0.00 mm
- net N$9: track 44.0 -> 73.1 mm, vias 2 -> 0
- net GND: track 141.7 -> 115.1 mm, vias 12 -> 22
- net N$8: track 43.7 -> 24.1 mm, vias 1 -> 0
- net VCC: track 70.4 -> 85.2 mm
- net N$16: track 44.1 -> 30.7 mm, vias 0 -> 1
- net N$11: track 38.2 -> 25.4 mm
- net N$17: track 52.8 -> 60.4 mm
- net N$19: track 78.9 -> 85.8 mm
- net N$10: track 75.1 -> 71.2 mm
- net N$1: track 15.7 -> 18.3 mm
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Other:
- board text added: "2.0.1"
- board text added: "MODE"
- board text added: "QC"
- board text added: "SYNCMAP"
- board text removed: "1.1.3"
- board text removed: "LIVE MAP"
