File: Eagle/Arduinoboy.sch (EAGLE design)
At the start: 20 parts

Commit message: update eagle files
Parts:
- removed R3: 2k, SparkFun-Resistors:RESISTORAXIAL-0.3
- removed U$1: GBA-LINK, David:GBA-LINK
- added U$4: GBA-LINK, Catskulls_link_port:GBA-LINK
Connections:
- removed net N$18: U$1.VCC, U$3.VIN
- removed net N$4: R3.2, S2.1, S2.2, U$3.D3
- new net N$20: S2.1, S2.2, U$3.D2
- new net PS2_CLK: U$3.D3, X1.5
- new net PS2_DATA: U$3.D7, X1.1
- net GND: now also S2.3, S2.4, U$4G$1.GND; no longer R3.1, U$1.GND
- net N$17: now also U$4G$1.SC; no longer U$1.SC, X1.5
- net N$21: now also U$4G$1.SO; no longer U$1.SO, X1.1
- net N$22: now also U$4G$1.SI; no longer U$1.SI
- net VCC: now also U$4G$1.SD, U$4G$1.VCC; no longer S2.3, S2.4
Other:
- moved on the sheet: S2
